File: Hardware/ST-Node-V0.1/LoRa-MCU.sch (KiCad schematic (older format))
At the start: 82 parts, among them J1 U.FL-R-SMT-1, SW1 RESET, U5 STM32WLxx_QFN48, U6 NX3L1T3157GM, U7 BGS13S4N9, U8 NX3L1T3157GM, X1 32MHz, X2 32.768KHz

Commit message: sch:  Swap couple of pins and fix a HW bug
Parts:
- removed AE1: Dual_Band_868/915, RF_Antenna:Texas_SWRA416_868MHz_915MHz, symbol Device:Antenna_Chip
- removed X1: 32MHz, Oscillator:Oscillator_SMD_Abracon_ASE-4Pin_3.2x2.5mm, symbol Oscillator:ASE-xxxMHz
- added AE1: Antenna, RF_Antenna:Texas_SWRA416_868MHz_915MHz, symbol Device:Antenna
- added X1: 32MHz, Oscillator:Oscillator_SMD_Abracon_ASE-4Pin_3.2x2.5mm, symbol node-lib-v1:TCXO-xxxMHz
- D3: renamed from D1; footprint (none) -> Inductor_SMD:L_0201_0603Metric
- FB1: footprint (none) -> Inductor_SMD:L_0603_1608Metric
- JP10: renamed from JP5; footprint (none) -> Jumper:SolderJumper-2_P1.3mm_Open_RoundedPad1.0x1.5mm
- JP11: renamed from JP6; footprint (none) -> Jumper:SolderJumper-3_P1.3mm_Bridged12_RoundedPad1.0x1.5mm_NumberLabels
- JP6, JP8: renamed from JP?; footprint (none) -> Jumper:SolderJumper-3_P1.3mm_Bridged12_RoundedPad1.0x1.5mm_NumberLabels
- JP7: renamed from JP4; footprint (none) -> Jumper:SolderJumper-3_P1.3mm_Bridged12_RoundedPad1.0x1.5mm_NumberLabels
- JP9: renamed from JP?; value PB12 -> INT; footprint (none) -> Jumper:SolderJumper-3_P1.3mm_Bridged12_RoundedPad1.0x1.5mm_NumberLabels
- L2: footprint (none) -> Inductor_SMD:L_0402_1005Metric
- L8: footprint (none) -> Inductor_SMD:L_0805_2012Metric
- R20: renamed from R9; footprint (none) -> Inductor_SMD:L_0402_1005Metric
- R21: renamed from R10; footprint (none) -> Inductor_SMD:L_0402_1005Metric
- R22: renamed from R11; footprint (none) -> Inductor_SMD:L_0402_1005Metric
- SW2: renamed from SW1; footprint (none) -> Button_Switch_SMD:SW_SPST_EVQP2
- renumbered C14 to C21, C15 to C22, C16 to C23, C17 to C24, C18 to C25, C19 to C26, C20 to C27, C21 to C28, C22 to C29, C23 to C30, C24 to C31, C25 to C32, C26 to C33, C27 to C34, C28 to C35, C29 to C36, C30 to C37, C31 to C38, C32 to C39, C33 to C40, C34 to C41, C35 to C42, C36 to C43, C37 to C44, C38 to C45, C39 to C46, C40 to C47, C41 to C48, C42 to C49, C43 to C50, C44 to C51, C45 to C52, C46 to C53, C47 to C54, C48 to C55, C49 to C56, C50 to C57, C51 to C58, C52 to C59, C53 to C60, C54 to C61, C55 to C62, C56 to C63, C57 to C64, C58 to C65, C59 to C66, J1 to J2, R12 to R23, R13 to R24, R14 to R25, R15 to R26, U6 to U10, U7 to U11, U8 to U12, U5 to U9
Connections:
- net labels added: PA8_INT1, PA8_INT2
- net labels removed: PA8, PB12_GLED
- wire segments 294 -> 295
Other:
- moved on the sheet: JP9

Commit message: sch, pcb: Improve pcb layout, swap sch pins
Parts:
- removed AE1: Antenna, RF_Antenna:Texas_SWRA416_868MHz_915MHz, symbol Device:Antenna
- removed L13: 8.7nH, Inductor_SMD:L_0402_1005Metric, symbol Device:L_Small
- added AE1: ANT_M620720, node-lib-v1:ANT_M620720, symbol node-lib-v1:ANT_M620720
- added C67: 5.0pF, Capacitor_SMD:C_0402_1005Metric, symbol Device:C_Small
- added C68: 3.6pF, Capacitor_SMD:C_0402_1005Metric, symbol Device:C_Small
- added R18: 0R, Resistor_SMD:R_0402_1005Metric, symbol Device:R_Small
- C21, C24, C41: MPN CC0603KRX5R7BB475 -> C1608X5R1C475K080AC
- C22, C23, C25, C26, C27, C42, C43, C61: footprint Capacitor_SMD:C_0603_1608Metric -> Capacitor_SMD:C_0402_1005Metric
- C30, C32: MPN GRM1555C1H6R8BA01 -> GRM1555C1H6R8BA01D
- C35: value 1pF -> DNM; DNM_MPN (none) -> CC0402BRNPO9BN1R0; MPN CC0402BRNPO9BN1R0 -> (none)
- C44: MPN CC0402BRNPO9BN6R8 -> GRM1555C1H6R8BA01D
- C58: value 33pF -> DNM; DNM_MPN (none) -> CC0402JRNPO9BN330; MPN CC0402JRNPO9BN330 -> (none)
- C59, C63: value 3.3pF -> DNM; DNM_MPN (none) -> CC0402BRNPO9BN3R3; MPN CC0402BRNPO9BN3R3 -> (none)
- C60, C64: value 100nF -> DNM; DNM_MPN (none) -> CC0402KRX7R7BB104; MPN CC0402KRX7R7BB104 -> (none)
- C62, C65, C66: footprint Capacitor_SMD:C_0603_1608Metric -> Capacitor_SMD:C_0402_1005Metric; MPN GRM1555C1H330GA01 -> CC0402JRNPO9BN330
- D3: footprint Inductor_SMD:L_0201_0603Metric -> Diode_SMD:D_0201_0603Metric
- FB1: MPN FCM1608KF-601T03 -> BLM18AG601SN1D
- JP10: footprint Jumper:SolderJumper-2_P1.3mm_Open_RoundedPad1.0x1.5mm -> Button_Switch_SMD:SW_SPST_B3U-1000P
- R20: value 10K -> DNM; DNM_MPN (none) -> AC0402JR-0710KL; MPN RC0402FR-0710KL -> (none)
- R22: MPN RC0402FR-0710KL -> AC0402JR-0710KL
- R26: MPN RC0402JR-070RL -> RC0402FR-070RL
- SW2: footprint Button_Switch_SMD:SW_SPST_EVQP2 -> node-lib-v1:EVQ-P2R02W; MPN KMR211GLFS -> EVQ-P2R02W
- U10, U12: footprint Package_DFN_QFN:DFN-6_1.3x1.2mm_P0.4mm -> node-lib-v1:6-XFDFN_SOT-886
- U11: footprint Package_CSP:LFCSP-8-1EP_3x2mm_P0.5mm_EP1.6x1.65mm -> node-lib-v1:RFSW_BGS13S4N9E6327XTSA1; MPN (none) -> BGS13S4N9E6327XTSA1
- U9: footprint Package_DFN_QFN:QFN-48-1EP_7x7mm_P0.5mm_EP5.6x5.6mm -> Package_DFN_QFN:QFN-48-1EP_7x7mm_P0.5mm_EP5.45x5.45mm_ThermalVias; MPN (none) -> STM32WLxx_QFN48
- X1: footprint Oscillator:Oscillator_SMD_Abracon_ASE-4Pin_3.2x2.5mm -> node-lib-v1:TCXO_NT2016SA-32M-END4263A
- X2: footprint Crystal:Crystal_SMD_TXC_7A-2Pin_5x3.2mm -> node-lib-v1:Crystal_SMD_NX2012SA_32.768KHz; MPN NX2012SA 32.768KHz EXS00A-MU00527 -> NX2012SA-32.768KHZ-EXS00A-MU00527
Connections:
- net labels added: SPI1_NSS_PA4
- net labels removed: PB8
- wire segments 295 -> 313
- no-connect marks 1 -> 2
Other:
- note added: "100nF"
- note added: "10K"
- note added: "1pF"
- note added: "33pF"
- note added: "C57 & C58 share \na common pad"
- note added: "P1"
- note added: "P2"
- moved on the sheet: C63, R26

Commit message: pcb, doc: Add final production files, add interaction PnP iBOM
dev: Add gitignore for KiCAD files


all: Delete unused media files
Parts:
- added R27: 0R, Resistor_SMD:R_0402_1005Metric, symbol Device:R_Small
- U9: footprint Package_DFN_QFN:QFN-48-1EP_7x7mm_P0.5mm_EP5.45x5.45mm_ThermalVias -> Package_DFN_QFN:QFN-48-1EP_7x7mm_P0.5mm_EP5.45x5.45mm
Connections:
- net VDDSMPS is gone; now on net VDDRF: C41.1, C43.1, U9.46 (VDDSMPS)
- net VDD: now also R27.2; no longer C25.1
- net VDDRF: now also C25.1, R27.1
- net RFI_P: now reaches C33.1, L5.2, U9.20 (RFI_P)
Other:
- note added: "28"
- note added: "Close to 46 (VDDSMPS)"
- moved on the sheet: C25, C27
Changed lines of the file:
@@
 F 0 "U9" H 3450 6167 60  0000 C CNB
 F 1 "STM32WLxx_QFN48" H 3450 6047 79  0000 C CNB
-F 2 "Package_DFN_QFN:QFN-48-1EP_7x7mm_P0.5mm_EP5.45x5.45mm_ThermalVias" H 3450 3550 60  0001 C CNN
+F 2 "Package_DFN_QFN:QFN-48-1EP_7x7mm_P0.5mm_EP5.45x5.45mm" H 3450 3550 60  0001 C CNN
 F 3 "https://www.st.com/resource/en/datasheet/stm32wle5jc.pdf" H 2350 5250 60  0001 C CNN
 F 4 "STM32WLxx_QFN48" H 2650 5950 50  0001 C CNN "MPN"
@@
 L Device:C C25
 U 1 1 5ED1DE4C
-P 1750 1275
-F 0 "C25" H 1865 1321 50  0000 L CNN
-F 1 "100nF" H 1825 1200 50  0000 L CNN
-F 2 "Capacitor_SMD:C_0402_1005Metric" H 1788 1125 50  0001 C CNN
-F 3 "~" H 1750 1275 50  0001 C CNN
-F 4 "CC0402KRX7R7BB104" H 1750 1275 50  0001 C CNN "MPN"
-	1    1750 1275
+P 2150 1275
+F 0 "C25" H 2265 1321 50  0000 L CNN
+F 1 "100nF" H 2225 1200 50  0000 L CNN
+F 2 "Capacitor_SMD:C_0402_1005Metric" H 2188 1125 50  0001 C CNN
+F 3 "~" H 2150 1275 50  0001 C CNN
+F 4 "CC0402KRX7R7BB104" H 2150 1275 50  0001 C CNN "MPN"
+	1    2150 1275
 	1    0    0    -1
 $EndComp
@@
 L Device:C C27
 U 1 1 5ED1E17D
-P 2125 1275
-F 0 "C27" H 2240 1321 50  0000 L CNN
-F 1 "100nF" H 2200 1200 50  0000 L CNN
-F 2 "Capacitor_SMD:C_0402_1005Metric" H 2163 1125 50  0001 C CNN
-F 3 "~" H 2125 1275 50  0001 C CNN
-F 4 "CC0402KRX7R7BB104" H 2125 1275 50  0001 C CNN "MPN"
-	1    2125 1275
+P 1725 1275
+F 0 "C27" H 1825 1275 50  0000 L CNN
+F 1 "100nF" H 1800 1200 50  0000 L CNN
+F 2 "Capacitor_SMD:C_0402_1005Metric" H 1763 1125 50  0001 C CNN
+F 3 "~" H 1725 1275 50  0001 C CNN
+F 4 "CC0402KRX7R7BB104" H 1725 1275 50  0001 C CNN "MPN"
+	1    1725 1275
 	1    0    0    -1
 $EndComp
@@
 	975  1075 975  1125
 Wire Wire Line
-	1750 1125 1750 1075
-Wire Wire Line
-	1750 1075 1350 1075
-Connection ~ 1350 1075
-Wire Wire Line
-	2125 1125 2125 1075
-Wire Wire Line
-	2125 1075 1750 1075
-Connection ~ 1750 1075
-Wire Wire Line
-	2125 1425 2125 1500
-Wire Wire Line
-	2125 1500 1750 1500
+	1725 1125 1725 1075
+Wire Wire Line
+	1725 1425 1725 1500
 Connection ~ 975  1500
 Wire Wire Line
@@
 Wire Wire Line
 	1350 1425 1350 1500
-Connection ~ 1350 1500
 Wire Wire Line
 	1350 1500 975  1500
-Wire Wire Line
-	1750 1425 1750 1500
-Connection ~ 1750 1500
-Wire Wire Line
-	1750 1500 1350 1500
 $Comp
 L Device:C C23
@@
 Text Notes 1150 1050 0    50   ~ 0
 44
-Text Notes 1875 1050 0    50   ~ 0
+Text Notes 1700 1050 0    50   ~ 0
 11
 Wire Wire Line
@@
 Wire Wire Line
 	4750 6450 4550 6450
-Text GLabel 9550 2075 2    59   Output ~ 12
+Text GLabel 11025 1700 0    59   Input ~ 12
 VDDSMPS
 $Comp
@@
 Text GLabel 15275 1725 1    59   Output ~ 12
 VDDPA
-Text GLabel 8325 2125 0    59   Input ~ 12
-VDDRF
 Connection ~ 9275 2075
 $Comp
@@
 	12450 1850 12350 1850
 Wire Wire Line
-	11025 1850 11150 1850
+	11125 1850 11150 1850
 Wire Wire Line
 	11025 1700 11150 1700
@@
 Text GLabel 12475 1700 2    59   Output ~ 12
 VDDPA
-Text GLabel 11025 1850 0    59   Input ~ 12
+Text GLabel 11125 1850 0    59   Input ~ 12
 VDDRF1V55
-Text GLabel 11025 1700 0    59   Input ~ 12
-VDDRF
 $Comp
 L node-lib-v1:NX3L1T3157GM U12
@@
 Text Notes 15100 6325 0    59   ~ 0
 P2
+Text Notes 8425 2050 0    59   ~ 0
+Close to 46 (VDDSMPS)
+Text GLabel 2150 950  1    59   Output ~ 12
+VDDRF
+Text Notes 2175 1075 0    50   ~ 0
+28
+Wire Wire Line
+	1725 1075 1350 1075
+Connection ~ 1350 1075
+Wire Wire Line
+	1725 1500 1350 1500
+Connection ~ 1350 1500
+$Comp
+L Device:R_Small R27
+U 1 1 5EF97B02
+P 1950 1075
+F 0 "R27" V 2025 1075 50  0000 C CNN
+F 1 "0R" V 1950 1075 50  0000 C CNN
+F 2 "Resistor_SMD:R_0402_1005Metric" H 1950 1075 50  0001 C CNN
+F 3 "~" H 1950 1075 50  0001 C CNN
+F 4 "RC0402FR-070RL" V 1950 1075 50  0001 C CNN "MPN"
+	1    1950 1075
+	0    1    1    0
+$EndComp
+Wire Wire Line
+	1850 1075 1725 1075
+Connection ~ 1725 1075
+Wire Wire Line
+	2150 950  2150 1075
+Wire Wire Line
+	2150 1425 2150 1500
+Wire Wire Line
+	2150 1500 1725 1500
+Connection ~ 1725 1500
+Wire Wire Line
+	2050 1075 2150 1075
+Connection ~ 2150 1075
+Wire Wire Line
+	2150 1075 2150 1125
+Text GLabel 9550 2075 2    59   Output ~ 12
+VDDSMPS
+Text Label 4850 8050 0    59   ~ 0
+RFI_P
+Text GLabel 8225 2075 0    59   Input ~ 12
+VDDRF
 $EndSCHEMATC
