File: Hardware/ST-Node-V0.1/ST-Node-V0.1.kicad_pcb (KiCad board)
At the start: 4 copper layers, 40.9 x 67.7 mm, 157 parts, among them J1 Debug, J2 U.FL-R-SMT-1, Q1 SI2323DS, Q2 2SC4213, SW1 SW_Push, SW2 RESET, U1 TPS22917DBV, U10 NX3L1T3157GM, U11 BGS13S4N9, U12 NX3L1T3157GM, U2 RP605Z283B, U3 TPS22917DBV, U4 TPS22917DBV, U5 MX25R1635, U6 LIS2DH12, U7 SHTC3, U8 ATECC608A-TNGLORAU, U9 STM32WLxx_QFN48, X1 32MHz, X2 32.768KHz

Commit message: pcb, doc: Add final production files, add interaction PnP iBOM
dev: Add gitignore for KiCAD files


all: Delete unused media files
Parts:
- added G***: LOGO, node-lib-v1:qr_azerimaker_11mm, B.Cu at (130.4, 72.4)
- added G***: LOGO, node-lib-v1:Icon_Battery_1000px, B.Cu at (147.8, 108.4)
- added G***: LOGO, node-lib-v1:Icon_Battery_1000px, B.Cu at (131.7, 107.8)
- added G***: LOGO, node-lib-v1:Logo_GN-4000px, B.Cu at (145.5, 71.1)
- added G***: LOGO, node-lib-v1:Logo_GN-4000px, F.Cu at (137.1, 74.1)
- added J3: Grove_I2C, Connector:NS-Tech_Grove_1x04_P2mm_Vertical, F.Cu at (125.7, 86.7)
- added R27: 0R, Resistor_SMD:R_0402_1005Metric, F.Cu at (133.2, 97.4)
- added REF**: OSHW-Logo2_9.8x8mm_SilkScreen, Symbol:OSHW-Logo2_9.8x8mm_SilkScreen, B.Cu at (139.7, 95.5)
- added REF**: ESD-Logo_6.6x6mm_SilkScreen, Symbol:ESD-Logo_6.6x6mm_SilkScreen, B.Cu at (147.8, 95.5)
- U9: footprint Package_DFN_QFN:QFN-48-1EP_7x7mm_P0.5mm_EP5.45x5.45mm_ThermalVias -> Package_DFN_QFN:QFN-48-1EP_7x7mm_P0.5mm_EP5.45x5.45mm
- moved R15 22.3 mm to (154.9, 108.9), turned to 270 degrees
- moved R14 21.7 mm to (153.9, 108.9), turned to 90 degrees
- moved R16 20.1 mm to (130.0, 124.9), turned to 90 degrees
- moved D1 16.3 mm to (148.0, 124.7)
- moved Q2 15.5 mm to (132.2, 124.9), turned to 0 degrees
- moved C43 13.5 mm to (144.0, 105.2), turned to 270 degrees
- moved C25 12.6 mm to (133.2, 99.3), turned to 180 degrees
- moved C41 12.4 mm to (142.8, 105.5), turned to 270 degrees
- moved U12 3.22 mm to (131.6, 90.7)
- moved TP3 2.61 mm to (130.6, 103.0)
- moved L5 2.53 mm to (142.7, 91.4)
- moved C33 2.50 mm to (143.2, 89.9)
- moved C35 2.46 mm to (142.7, 88.5)
- moved C20 2.44 mm to (150.3, 99.5)
- moved C37 2.44 mm to (150.3, 98.5)
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Connections:
- net Net-(C33-Pad1) renamed /LoRa MCU/RFI_P
- AE1 pad 2: (no net) -> Net-(AE1-Pad2)
- C25 pad 1: VDD -> VDDRF
- D2 pad 2: (no net) -> Net-(D2-Pad2)
- J1 pad 9: (no net) -> Net-(J1-Pad9)
- U7 pad 5: (no net) -> Net-(U7-Pad5)
- U9 pad 12: FE_CTRL3 -> /Peripherals/FlashCS
- U9 pad 27: (no net) -> Net-(U9-Pad27)
- U9 pad 6: /Peripherals/FlashCS -> FE_CTRL3
Routing:
- net GND: track 14.4 -> 175.5 mm, vias 23 -> 244
- net VDD: track 28.6 -> 179.8 mm, vias 12 -> 29
- net /LoRa MCU/I2C1_SCL: track 0.00 -> 69.9 mm, vias 0 -> 4
- net NRST: track 0.00 -> 69.3 mm, vias 0 -> 3
- net /LoRa MCU/USART2_TxD: track 0.00 -> 54.2 mm, vias 0 -> 2
- net /LoRa MCU/I2C1_SDA: track 0.00 -> 53.2 mm, vias 0 -> 3
- net /Peripherals/VCC_SENSORS: track 0.00 -> 51.7 mm, vias 0 -> 6
- net /LoRa MCU/USART2_RxD: track 0.00 -> 50.5 mm, vias 0 -> 2
- net /LoRa MCU/I2C2_SDA: track 0.00 -> 48.5 mm, vias 0 -> 4
- net VDDRF: track 0.00 -> 46.7 mm, vias 0 -> 5
- net /LoRa MCU/PB3: track 0.00 -> 45.9 mm, vias 0 -> 2
- net /LoRa MCU/I2C2_SCL: track 0.00 -> 44.6 mm, vias 0 -> 4
- net FE_CTRL1: track 0.00 -> 44.1 mm, vias 0 -> 4
- net FE_CTRL2: track 0.00 -> 38.9 mm, vias 0 -> 3
- net VDDRF1V55: track 1.43 -> 38.5 mm, vias 0 -> 5
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- added copper zone on F.Cu, net Net-(AE1-Pad1)
- added copper zone on In2.PWR, net Net-(BH2-Pad1)
Other:
- outline, holes or cut-outs redrawn
- net class 100Ohm added: clearance 0.1524, trace_width 0.1397, via_dia 0.8, via_drill 0.4
- net class Default: trace_width 0.1524 -> 0.1397
- board text added: "1.5V-AA"
- board text added: "Accel."
- board text added: "Grove"
- board text added: "X"
- board text added: "Y"
- board text added: "Z"
- board text added: "v.0.1"
- board text removed: "Accelerometer"
- board text removed: "Generic Node"
