File: Hardware/ST-Node-V0.1/ST-Node-V0.1.sch (KiCad schematic (older format))
At the start: 0 parts

Commit message: pcb, doc: Add final production files, add interaction PnP iBOM
dev: Add gitignore for KiCAD files


all: Delete unused media files
Changed lines of the file:
@@
 F7 "USART2_TxD" O L 5575 2200 59
 F8 "USART2_RxD" I L 5575 2275 59
-F9 "PA4" B R 7500 2125 59
+F9 "SPI1_NSS_PA4" B R 7500 2125 59
 F10 "PB12" B L 5575 1200 59
 F11 "PC13" B R 7500 2750 59
