File: Hardware/pcb-bolink-batteryHolder/pcb-bolink-batteryHolder.sch (KiCad schematic (older format))
At the start: 44 parts, among them J1 S1001-46R, J2 JST-PH, J3 S1001-46R, J4 RF_Shield_One_Piece, J5 S1001-46R, J6 S1001-46R, Q1 CEN2321A, U1 TPS22917DBV, U2 TPS3839G25, U3 TPS22917DBV, U4 RP605Z283B

Commit message: pcb,sch: Add V0.2 HW design with external battery holder
Parts:
- removed C1, C4, C5: 100uF, Capacitor_SMD:C_1206_3216Metric, symbol Device:C
- removed C10, C7, C9: 100nF, Capacitor_SMD:C_0402_1005Metric, symbol Device:C
- removed C11, C3, C6, C8: 1uF, Capacitor_SMD:C_0402_1005Metric, symbol Device:C
- removed C12: 22uF, Capacitor_SMD:C_0603_1608Metric, symbol Device:C
- removed C2: 10nF, Capacitor_SMD:C_0402_1005Metric, symbol Device:C_Small
- removed D1: PESD5V0S1BA, Diode_SMD:D_SOD-323, symbol Device:D_TVS_ALT
- removed F1: PTC 13V 1A, Fuse:Fuse_1210_3225Metric_Castellated, symbol Device:Polyfuse
- removed FID1, FID2, FID3, FID4, FID5, FID6: Fiducial, Fiducial:Fiducial_0.5mm_Mask1.5mm, symbol Mechanical:Fiducial
- removed H1, H2: MountingHole, MountingHole:MountingHole_2.5mm, symbol Mechanical:MountingHole
- removed J1, J3, J5, J6: S1001-46R, node-lib-v1:RF_Shield_Clip_S1001-46R, symbol Connector:Conn_01x01_Female
- removed J2: JST-PH, Connector_JST:JST_PH_B2B-PH-SM4-TB_1x02-1MP_P2.00mm_Vertical, symbol Connector_Generic:Conn_01x02
- removed J4: RF_Shield_One_Piece, node-lib-v1:RF_Shield_SnapOn_30x20mm_w_Cutout_n_GND_Pads, symbol Device:RF_Shield_One_Piece
- removed L1: 2.2uH, node-lib-v1:L_HPC4012TF-2R2M, symbol Device:L_Core_Ferrite
- removed N1: BoLink-16174563, node-lib-v1:BoLink_704025, symbol Mechanical:Housing
- removed Q1: CEN2321A, Package_TO_SOT_SMD:SOT-23, symbol Device:Q_PMOS_GSD
- removed R1: 10K, Resistor_SMD:R_0402_1005Metric, symbol Device:R
- removed R2, R3, R4: 100K, Resistor_SMD:R_0402_1005Metric, symbol Device:R
- removed TP1: VIN, TestPoint:TestPoint_Pad_D1.5mm, symbol Connector:TestPoint_Probe
- removed TP2: VBAT, TestPoint:TestPoint_Pad_D1.5mm, symbol Connector:TestPoint_Probe
- removed TP3: VBAT_READ_EN, TestPoint:TestPoint_Pad_D1.5mm, symbol Connector:TestPoint_Probe
- removed TP4: VBAT_ADC, TestPoint:TestPoint_Pad_D1.5mm, symbol Connector:TestPoint_Probe
- removed TP5: VCC, TestPoint:TestPoint_Pad_D1.5mm, symbol Connector:TestPoint_Probe
- removed U1, U3: TPS22917DBV, Package_TO_SOT_SMD:SOT-23-6, symbol Power_Management:TPS22917DBV
- removed U2: TPS3839G25, Package_TO_SOT_SMD:SOT-23, symbol Power_Supervisor:TPS3839DBZ
- removed U4: RP605Z283B, node-lib-v1:WLCSP-20-P3_1.994x1.609mm_Layout5x4_P0.4mm, symbol node-lib-v1:RP605Zx
- added BT1, BT2: 2xPN57, node-lib-v1:keystone-PN57, symbol Device:Battery_Cell
- added BTclip1: PN69, node-lib-v1:Keystone_69_clip, symbol Mechanical:DIN_Rail_Adapter
- added J1: Batt-, TestPoint:TestPoint_Keystone_5019_Minature, symbol Connector_Generic:Conn_01x01
- added J2: Batt+, TestPoint:TestPoint_Keystone_5019_Minature, symbol Connector_Generic:Conn_01x01
- added J3: MOLEX PicoBlade 1.25mm, Connector_Molex:Molex_PicoBlade_53398-0271_1x02-1MP_P1.25mm_Vertical, symbol Connector_Generic:Conn_01x02
Connections:
- net labels added: VCC
- net labels removed: +2V8, +BATT, LS1_SENSORS_EN, LS2_FLASH_EN, VBAT_ADC, VBAT_READ_EN, VCC_FLASH, VCC_SENSORS, Vin
- wire segments 139 -> 17
- no-connect marks 2 -> 0
Other:
- note removed: "- Output: Vin/3 (division ratio)\n- Supply Current: 100nA\n- Settling time: ≥ 10ms"
- note removed: "- Vin: 1.8 - 5.5V\n- Vout: 1.6 - 5.2V\n- Iout: 300 mA\n- Iq: 300 nA\n- Output V: ±1.5%\n- w/ auto-discharge"
- note removed: "Buck-Boost Converter"
- note removed: "EMI Shield Can & Clips"
- note removed: "Enclosure & Logos"
- note removed: "Input ESD, Reverse Polarity \n& Short-Circuit Protection"
- note removed: "Load Switch 1 \nSensors & Secure Element"
- note removed: "Load Switch 2 - Flash"
- note removed: "Mounting Holes & Fiducials"
- note removed: "Voltage Supervisor\nVcut-off = 2.325V"
- note removed: "~Battery Monitor (BM):"
- note removed: "~Buck-Boost Specs:"
